File: hardware/picotouch_grid/picotouch_grid.kicad_pcb (KiCad board)
At the start: 2 copper layers, 180 x 110 mm, 170 parts, among them J1 TRRS, J2 TRRS, J3 TRRS, U1 Pico, U2 TS20, U3 TS20, U5 H11L1

Commit message: update readme
Parts:
- DISP1: footprint todbot_stuff:OLED-TH_under_L27.8-W27.2-P2.54_C9900033791 -> todbot_stuff:OLED-TH_under_fixed_L27.8-W27.2-P2.54_C9900033791
- TP1, TP2: footprint todbot_eagle2023:TOUCHPAD_KEY_0.5IN_LEDHOLE -> todbot_eagle2023:TOUCHPAD_KEY_0.5IN_LEDHOLE_OFFSET
- TP45, TP46: footprint todbot_stuff:Pad-CapacitiveTouch-SparkFun-10x5mm-roundrect -> SparkFun-Switch:Pad-CapacitiveTouch
- moved LED1 5.33 mm to (49.5, 71.4)
- moved LED2 5.27 mm to (66.0, 71.4)
Other:
- outline, holes or cut-outs redrawn
