File: hardware/picotouch_grid/picotouch_grid.kicad_sch (KiCad schematic)
At the start: 170 parts, among them J1 TRRS, J2 TRRS, J3 TRRS, U1 Pico, U2 TS20, U3 TS20, U5 H11L1

Commit message: update readme
Parts:
- DISP1: footprint easyeda2kicad:OLED-TH_L27.8-W27.2-P2.54_C9900033791 -> todbot_stuff:OLED-TH_under_fixed_L27.8-W27.2-P2.54_C9900033791
- U1: footprint RPi_Pico:RPi_Pico_SMD_TH -> todbot_RPI_Pico:RPi_Pico_SMD
Connections:
- no-connect marks 16 -> 19
Changed lines of the file:
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@@
 	)
 	(no_connect
+		(at 44.45 160.02)
+	)
+	(no_connect
 		(at 212.09 264.16)
 	)
@@
 	)
 	(no_connect
+		(at 44.45 185.42)
+	)
+	(no_connect
 		(at 104.14 59.69)
 	)
+	(no_connect
+		(at 44.45 132.08)
+	)
 	(wire
 		(pts
@@
 			)
 		)
-		(property "Footprint" "easyeda2kicad:OLED-TH_L27.8-W27.2-P2.54_C9900033791"
+		(property "Footprint" "todbot_stuff:OLED-TH_under_fixed_L27.8-W27.2-P2.54_C9900033791"
 			(at 34.29 91.44 0)
 			(effects
@@
 			)
 		)
-		(property "Footprint" "RPi_Pico:RPi_Pico_SMD_TH"
+		(property "Footprint" "todbot_RPI_Pico:RPi_Pico_SMD"
 			(at 86.36 63.5 90)
 			(effects
